File: switch.kicad_sch (KiCad schematic)
At the start: 2 parts, among them SW101 SW_Push

Commit message: Update README.md
Other:
- title: (none) -> CHORD ZERO
Changed lines of the file:
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@@
 (kicad_sch (version 20211123) (generator eeschema)
   (paper "A5")
+  (title_block
+    (title "CHORD ZERO")
+    (date "2022-08-17")
+    (rev "1")
+    (comment 3 "License: CERN Open Hardware Licence Version 2 - Strongly Reciprocal")
+    (comment 4 "Designed by: Simon Hengel")
+  )
   (wire (pts (xy 92.71 60.96) (xy 96.52 60.96))
     (stroke (width 0) (type default) (color 0 0 0 0))
